File: Hardware/PCB/yash/yash.kicad_sch (KiCad schematic)
At the start: 45 parts

Commit message: Redo guard ring as redundant tracks
Parts:
- C1: value (none) -> 1nF (PP); footprint (none) -> ao_tht:C_Rect_L7.2mm_W4.5mm_P5.00mm_FKS2_FKP2_MKS2_MKP2
- C2: value (none) -> 470pF; footprint (none) -> ao_tht:C_Disc_D3.0mm_W1.6mm_P2.50mm
- C3: value (none) -> 470nF; footprint (none) -> ao_tht:C_Rect_L7.2mm_W4.5mm_P5.00mm_FKS2_FKP2_MKS2_MKP2
- C4, C6, C7: value (none) -> 100nF; footprint (none) -> ao_tht:C_Disc_D3.0mm_W1.6mm_P2.50mm
- C5, C8: value (none) -> 10uF; footprint (none) -> ao_tht:CP_Radial_D6.3mm_P2.50mm
- D1: value (none) -> LED_green; footprint (none) -> ao_tht:LED_D5.0mm
- D2, D3: value (none) -> 1N4148; footprint (none) -> ao_tht:D_DO-35_SOD27_P7.62mm_Horizontal
- D5, D6: value (none) -> 1N5817; footprint (none) -> ao_tht:D_DO-41_SOD81_P10.16mm_Horizontal
- GRAF1: value (none) -> Holes; footprint (none) -> yash:yash_panel_holes
- J1, J2, J4: value (none) -> AudioJack2; footprint (none) -> ao_tht:Jack_6.35mm_PJ_629HAN_slots
- J10, J7: value (none) -> 2_pin_Molex_header; footprint (none) -> ao_tht:Molex_KK-254_AE-6410-02A_1x02_P2.54mm_Vertical
- J11, J8: value (none) -> 2_pin_Molex_connector; footprint (none) -> ao_tht:Molex_KK-254_AE-6410-02A_1x02_P2.54mm_Vertical
- J3: value (none) -> AudioJack2_SwitchT; footprint (none) -> ao_tht:Jack_6.35mm_PJ_629HAN_slots
- J5: value (none) -> 3_pin_Molex_header; footprint (none) -> ao_tht:Molex_KK-254_AE-6410-03A_1x03_P2.54mm_Vertical
- J6: value (none) -> 3_pin_Molex_connector; footprint (none) -> ao_tht:Molex_KK-254_AE-6410-03A_1x03_P2.54mm_Vertical
- J9: value (none) -> Synth_power_2x5; footprint (none) -> ao_tht:Power_Header
- Q1: value (none) -> 2N3904; footprint (none) -> ao_tht:TO-92_Inline_Wide
- R1: value (none) -> 1k; footprint (none) -> ao_tht:R_Axial_DIN0207_L6.3mm_D2.5mm_P10.16mm_Horizontal
- R10, R12: value (none) -> 2.2k; footprint (none) -> ao_tht:R_Axial_DIN0207_L6.3mm_D2.5mm_P10.16mm_Horizontal
- R2, R8: value (none) -> 100k; footprint (none) -> ao_tht:R_Axial_DIN0207_L6.3mm_D2.5mm_P10.16mm_Horizontal
- R3: value (none) -> RL; footprint (none) -> ao_tht:R_Axial_DIN0207_L6.3mm_D2.5mm_P10.16mm_Horizontal
- R4: value (none) -> 5.6k; footprint (none) -> ao_tht:R_Axial_DIN0207_L6.3mm_D2.5mm_P10.16mm_Horizontal
- R5: value (none) -> 4.7k; footprint (none) -> ao_tht:R_Axial_DIN0207_L6.3mm_D2.5mm_P10.16mm_Horizontal
- R6: value (none) -> 10k; footprint (none) -> ao_tht:R_Axial_DIN0207_L6.3mm_D2.5mm_P10.16mm_Horizontal
- R7: value (none) -> 1.8k; footprint (none) -> ao_tht:R_Axial_DIN0207_L6.3mm_D2.5mm_P10.16mm_Horizontal
- R9: value (none) -> 2.7k; footprint (none) -> ao_tht:R_Axial_DIN0207_L6.3mm_D2.5mm_P10.16mm_Horizontal
- RV1: value (none) -> 100k; footprint (none) -> ao_tht:Potentiometer_Alpha_16mm_Single_Vertical
- RV2: value (none) -> 1M; footprint (none) -> ao_tht:Potentiometer_Alpha_16mm_Single_Vertical
- SW1: value (none) -> SW_SPDT; footprint (none) -> ao_tht:SPDT-toggle-switch-1M-series
- TP1: value (none) -> -12V; footprint (none) -> ao_tht:TestPoint_THTPad_D1.5mm_Drill0.7mm
- TP2: value (none) -> +12V; footprint (none) -> ao_tht:TestPoint_THTPad_D1.5mm_Drill0.7mm
- TP3: value (none) -> GND; footprint (none) -> ao_tht:TestPoint_THTPad_1.5x1.5mm_Drill0.7mm
- U2: value (none) -> 4093; footprint (none) -> ao_tht:DIP-14_W7.62mm_Socket_LongPads

Commit message: CW not CCW, put LED on correct side of PCB
Parts:
- U1: value (none) -> LF398; footprint (none) -> ao_tht:DIP-8_W7.62mm_Socket_LongPads
Connections:
- net CLKFR_CCW renamed CLKFR_CW
Other:
- note added: "Added S&H/T&H switch"
Changed lines of the file:
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@@
+    (effects (font (size 1.27 1.27)) (justify left bottom))
+  )
+  (text "Added S&H/T&H switch" (at 106.68 60.96 0)
     (effects (font (size 1.27 1.27)) (justify left bottom))
   )
@@
     (effects (font (size 1.27 1.27)) (justify left bottom))
   )
-  (global_label "CLKFR_CCW" (shape input) (at 185.42 133.35 180) (fields_autoplaced)
+  (global_label "CLKFR_CW" (shape input) (at 185.42 133.35 180) (fields_autoplaced)
     (effects (font (size 1.27 1.27)) (justify right))
-    (property "Intersheet References" "${INTERSHEET_REFS}" (id 0) (at 172.2101 133.2706 0)
+    (property "Intersheet References" "${INTERSHEET_REFS}" (id 0) (at 173.4801 133.2706 0)
       (effects (font (size 1.27 1.27)) (justify right) hide)
     )
@@
     )
   )
-  (global_label "CLKFR_CCW" (shape output) (at 54.61 121.92 0) (fields_autoplaced)
+  (global_label "CLKFR_CW" (shape output) (at 54.61 121.92 0) (fields_autoplaced)
     (effects (font (size 1.27 1.27)) (justify left))
-    (property "Intersheet References" "${INTERSHEET_REFS}" (id 0) (at 67.8199 121.8406 0)
+    (property "Intersheet References" "${INTERSHEET_REFS}" (id 0) (at 66.5499 121.8406 0)
       (effects (font (size 1.27 1.27)) (justify left) hide)
     )
@@
     (in_bom yes) (on_board yes)
     (property "Reference" "U1" (id 0) (at 195.58 45.72 0))
-    (property "Value" "" (id 1) (at 195.58 48.26 0))
-    (property "Footprint" "" (id 2) (at 186.69 53.34 0)
-      (effects (font (size 1.27 1.27)) hide)
-    )
+    (property "Value" "LF398" (id 1) (at 195.58 48.26 0))
+    (property "Footprint" "ao_tht:DIP-8_W7.62mm_Socket_LongPads" (id 2) (at 186.69 53.34 0)
+      (effects (font (size 1.27 1.27)) hide)
+    )

Commit message: Post fab updates
Parts:
- C1: value 1nF (PP) -> (none); footprint ao_tht:C_Rect_L7.2mm_W4.5mm_P5.00mm_FKS2_FKP2_MKS2_MKP2 -> (none); SKU (none) -> FKP2G011001D00HSSD; Vendor Tayda -> DigiKey
- C2: value 470pF -> (none); footprint ao_tht:C_Disc_D3.0mm_W1.6mm_P2.50mm -> (none)
- C3: value 470nF -> (none); footprint ao_tht:C_Rect_L7.2mm_W4.5mm_P5.00mm_FKS2_FKP2_MKS2_MKP2 -> (none); SKU (none) -> A-568
- C4, C6, C7: value 100nF -> (none); footprint ao_tht:C_Disc_D3.0mm_W1.6mm_P2.50mm -> (none)
- C5, C8: value 10uF -> (none); footprint ao_tht:CP_Radial_D6.3mm_P2.50mm -> (none)
- D1: value LED_green -> (none); footprint ao_tht:LED_D5.0mm -> (none)
- D2, D3: value 1N4148 -> (none); footprint ao_tht:D_DO-35_SOD27_P7.62mm_Horizontal -> (none)
- D5, D6: value 1N5817 -> (none); footprint ao_tht:D_DO-41_SOD81_P10.16mm_Horizontal -> (none)
- GRAF1: value Holes -> (none); footprint yash:yash_panel_holes -> (none)
- J1, J2, J4: value AudioJack2 -> (none); footprint ao_tht:Jack_6.35mm_PJ_629HAN_slots -> (none); SKU (none) -> A-1121; Vendor (none) -> Tayda
- J10, J7: value 2_pin_Molex_header -> (none); footprint ao_tht:Molex_KK-254_AE-6410-02A_1x02_P2.54mm_Vertical -> (none)
- J11, J8: value 2_pin_Molex_connector -> (none); footprint ao_tht:Molex_KK-254_AE-6410-02A_1x02_P2.54mm_Vertical -> (none)
- J3: value AudioJack2_SwitchT -> (none); footprint ao_tht:Jack_6.35mm_PJ_629HAN_slots -> (none); SKU (none) -> A-1121; Vendor (none) -> Tayda
- J5: value 3_pin_Molex_header -> (none); footprint ao_tht:Molex_KK-254_AE-6410-03A_1x03_P2.54mm_Vertical -> (none)
- J6: value 3_pin_Molex_connector -> (none); footprint ao_tht:Molex_KK-254_AE-6410-03A_1x03_P2.54mm_Vertical -> (none)
- J9: value Synth_power_2x5 -> (none); footprint ao_tht:Power_Header -> (none)
- Q1: value 2N3904 -> (none); footprint ao_tht:TO-92_Inline_Wide -> (none)
- R1: value 1k -> (none); footprint ao_tht:R_Axial_DIN0207_L6.3mm_D2.5mm_P10.16mm_Horizontal -> (none)
- R10, R12: value 2.2k -> (none); footprint ao_tht:R_Axial_DIN0207_L6.3mm_D2.5mm_P10.16mm_Horizontal -> (none)
- R2, R8: value 100k -> (none); footprint ao_tht:R_Axial_DIN0207_L6.3mm_D2.5mm_P10.16mm_Horizontal -> (none)
- R3: value RL -> (none); footprint ao_tht:R_Axial_DIN0207_L6.3mm_D2.5mm_P10.16mm_Horizontal -> (none)
- R4: value 5.6k -> (none); footprint ao_tht:R_Axial_DIN0207_L6.3mm_D2.5mm_P10.16mm_Horizontal -> (none)
- R5: value 4.7k -> (none); footprint ao_tht:R_Axial_DIN0207_L6.3mm_D2.5mm_P10.16mm_Horizontal -> (none)
- R6: value 10k -> (none); footprint ao_tht:R_Axial_DIN0207_L6.3mm_D2.5mm_P10.16mm_Horizontal -> (none)
- R7: value 1.8k -> (none); footprint ao_tht:R_Axial_DIN0207_L6.3mm_D2.5mm_P10.16mm_Horizontal -> (none)
- R9: value 2.7k -> (none); footprint ao_tht:R_Axial_DIN0207_L6.3mm_D2.5mm_P10.16mm_Horizontal -> (none)
- RV1: value 100k -> (none); footprint ao_tht:Potentiometer_Alpha_16mm_Single_Vertical -> (none); SKU (none) -> A-1984
- RV2: value 1M -> (none); footprint ao_tht:Potentiometer_Alpha_16mm_Single_Vertical -> (none); SKU (none) -> A-1658
- SW1: value SW_SPDT -> (none); footprint ao_tht:SPDT-toggle-switch-1M-series -> (none)
- TP1: value -12V -> (none); footprint ao_tht:TestPoint_THTPad_D1.5mm_Drill0.7mm -> (none)
- TP2: value +12V -> (none); footprint ao_tht:TestPoint_THTPad_D1.5mm_Drill0.7mm -> (none)
- TP3: value GND -> (none); footprint ao_tht:TestPoint_THTPad_1.5x1.5mm_Drill0.7mm -> (none)
- U1: value LF398 -> (none); footprint ao_tht:DIP-8_W7.62mm_Socket_LongPads -> (none); SKU (none) -> LF398AN/NOPB-ND; Vendor (none) -> Digi-Key
- U2: value 4093 -> (none); footprint ao_tht:DIP-14_W7.62mm_Socket_LongPads -> (none); SKU (none) -> A-554; Vendor (none) -> Tayda
